Commit message: Update delta_robot.urdf

File: ch3/delta_robot/urdf/delta_robot.urdf (robot description, URDF)
Before this commit: robot delta_robot, 18 links, 17 joints
Links:
- removed link con1
- removed link con13
- removed link con2
- removed link con23
- removed link con3
- removed link con33
- removed link link_0
- removed link lleg_1
- removed link lleg_12
- removed link lleg_2
- removed link lleg_22
- removed link lleg_3
- removed link lleg_32
- removed link low_base
- removed link uleg_1
- removed link uleg_2
- removed link uleg_3
- removed link world
- added link arm_1; visual box size=0.300 0.02 0.02
- added link arm_2; visual box size=0.300 0.02 0.02
- added link arm_3; visual box size=0.300 0.02 0.02
- added link base_link; visual cylinder length=0.02 radius=0.180
- added link down_arm_1; visual box size=0.800 0.02 0.02
- added link down_arm_2; visual box size=0.800 0.02 0.02
- added link down_arm_3; visual box size=0.800 0.02 0.02
- added link tool0; visual cylinder length=0.02 radius=0.100
Joints:
- removed joint base
- removed joint con13_lleg_1
- removed joint con23_lleg_2
- removed joint con2_lleg_1
- removed joint con2_lleg_2
- removed joint con2_lleg_3
- removed joint con33_lleg_3
- removed joint con_lleg_1
- removed joint con_lleg_2
- removed joint con_lleg_3
- removed joint link_0_JOINT_1
- removed joint link_0_JOINT_2
- removed joint link_0_JOINT_3
- removed joint lleg1_base
- removed joint uleg1_con
- removed joint uleg2_con
- removed joint uleg3_con
- added joint base_to_arm_1: type revolute, parent base_link, child arm_1, origin xyz=0 -0.180 0 rpy=0 0 -1.5708, axis 0 1 0, limit lower=-1.5708 upper=1.5708 effort=1000.0 velocity=0.5
- added joint base_to_arm_2: type revolute, parent base_link, child arm_2, origin xyz=0.155885 0.09 0 rpy=0 0 0.5236, axis 0 1 0, limit lower=-1.5708 upper=1.5708 effort=1000.0 velocity=0.5
- added joint base_to_arm_3: type revolute, parent base_link, child arm_3, origin xyz=-0.155885 0.09 0 rpy=0 0 2.618, axis 0 1 0, limit lower=-1.5708 upper=1.5708 effort=1000.0 velocity=0.5
- added joint down_arm_1_to_arm_1: type revolute, parent arm_1, child down_arm_1, origin xyz=0.300 0 0 rpy=0 1.5708 0, axis 0 1 0, limit lower=-1.5708 upper=1.5708 effort=1000.0 velocity=0.5
- added joint down_arm_2_to_arm_2: type revolute, parent arm_2, child down_arm_2, origin xyz=0.300 0 0 rpy=0 1.5708 0, axis 0 1 0, limit lower=-1.5708 upper=1.5708 effort=1000.0 velocity=0.5
- added joint down_arm_3_to_arm_3: type revolute, parent arm_3, child down_arm_3, origin xyz=0.300 0 0 rpy=0 1.5708 0, axis 0 1 0, limit lower=-1.5708 upper=1.5708 effort=1000.0 velocity=0.5
- added joint tool0_to_down_arm_1: type revolute, parent down_arm_1, child tool0, origin xyz=0.800 0 0 rpy=0 1.5708 0, axis 0 1 0, limit lower=-1.5708 upper=1.5708 effort=1000.0 velocity=0.5
